Commit message: Added infrared sensor

File: hector_quadrotor_description/urdf/quadrotor_hokuyo_utm30lx.gazebo.xacro (robot description, xacro)
@@ -3,3 +3,13 @@
     <xacro:include filename="$(find hector_quadrotor_description)/urdf/quadrotor_hokuyo_utm30lx.urdf.xacro" />
     <xacro:include filename="$(find hector_quadrotor_gazebo)/urdf/quadrotor_plugins.gazebo.xacro" />
+<!--    <link name = "link"></link>
+    <include>
+        <uri>model://infrared_sensor</uri>
+        <pose>0 0 0.15 -1.57 0 0</pose>
+    </include>
+    <joint name = "infrared_joint" type = "fixed">
+        <child>infrared_sensor::link</child>
+        <parent>quadrotor::link</parent>
+    </joint>
+-->
 </robot>
