Commit message: Added sensors back

File: hector_quadrotor_description/urdf/quadrotor_hokuyo_infrared.urdf.xacro (robot description, xacro)
@@ -18,6 +18,6 @@
     <!-- Infrared sensor -->
     <xacro:include filename="$(find hector_sensors_description)/urdf/infrared_sensor.urdf.xacro" />
-    <xacro:infrared_sensor name="bottom_infr" parent="base_link" ros_topic="/infrared_scan" update_rate="40" ray_count="1081" min_angle="-135" max_angle="135">
-      <origin xyz="0.05 0.0 -0.06" rpy="0 -1.57 0"/>
+    <xacro:infrared_sensor name="bottom_infr" parent="base_link" ros_topic="/infrared_scan" update_rate="40" ray_count="1081" min_angle="89" max_angle="91">
+      <origin xyz="0.0 0.0 -0.05" rpy="0 0 -1.57"/>
     </xacro:infrared_sensor>
 </robot>

Commit message: Fixed infrared position

File: hector_quadrotor_description/urdf/quadrotor_hokuyo_infrared.urdf.xacro (robot description, xacro)
@@ -19,5 +19,5 @@
     <xacro:include filename="$(find hector_sensors_description)/urdf/infrared_sensor.urdf.xacro" />
     <xacro:infrared_sensor name="bottom_infr" parent="base_link" ros_topic="/infrared_scan" update_rate="40" ray_count="1081" min_angle="89" max_angle="91">
-      <origin xyz="0.0 0.0 -0.05" rpy="0 0 -1.57"/>
+      <origin xyz="0.05 0.0 -0.04" rpy="-1.57 0 -1.57"/>
     </xacro:infrared_sensor>
 </robot>
